File: Ganglion_01.kicad_pcb (KiCad board)
At the start: 4 copper layers, 45 x 35 mm, 122 parts, among them J1 Conn_01x03, J2 Conn_01x03, SW1 CJS1200, SW2 CJS1200, SW5 SPDT, SW6 TACT_SWITCH, U1 MCP6V31U, U10 NCP300, U11 NCP551, U12 AD5621, U14 MCP6V13T, U15 MCP6001, U16 SN74LVC1G32, U17 LIS2DE12, U18 74LVC1G66, U2 AD8237, U21 74LVC1G66, U22 74LVC1G66, U23 74LVC2G00, U25 MCP6V31U, U26 MCP6V31U, U28 TPD4E1B06, U29 TPD4E1B06, U3 AD8237, U6 LM7332, U7 MCP3912, U8 ESP32-S3-MINI-1, U9 NCP551, Y1 Crystal_Small

Commit message: BOM cleanup
Parts:
- added C47: 22uF, Capacitor_SMD:C_0603_1608Metric, F.Cu at (136.2, 57.5)
- added C48: 22uF, Capacitor_SMD:C_0603_1608Metric, F.Cu at (137.8, 57.5)
- C38, C43: value 18pF -> 33pF
- R6: value R -> 1K
- U11, U9: value NCP551 -> TLV75730PDBVR
- U14: value MCP6V13T -> MCP6V31T
Routing:
- net Net-(U8-GPIO0/BOOT): track 15.5 -> 20.2 mm
- net VDD: track 42.1 -> 45.3 mm
- net GNDA: track 180.7 -> 183.9 mm
