File: Ganglion_01.kicad_sch (KiCad schematic)
At the start: 43 parts, among them J1 Conn_01x03, J2 Conn_01x03, SW1 CJS1200, SW2 CJS1200, U2 AD8237, U25 MCP6V31U, U3 AD8237, U6 LM7332, U7 MCP3912, Y1 Crystal_Small

Commit message: BOM cleanup
Parts:
- C38, C43: value 18pF -> 33pF; MPN GJM0335C1E180GB01D -> CL10C330JB8NNNC; SPN 490-14486-1-ND -> 1276-1070-1-ND
Changed lines of the file:
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@@
 			)
 		)
-		(property "Value" "18pF"
+		(property "Value" "33pF"
 			(at 285.75 161.29 0)
 			(effects
@@
 			)
 		)
-		(property "MPN" "GJM0335C1E180GB01D"
+		(property "MPN" "CL10C330JB8NNNC"
 			(at 280.67 163.83 0)
 			(effects
@@
 			)
 		)
-		(property "SPN" "490-14486-1-ND"
+		(property "SPN" "1276-1070-1-ND"
 			(at 280.67 163.83 0)
 			(effects
@@
 			)
 		)
-		(property "Value" "18pF"
+		(property "Value" "33pF"
 			(at 302.895 161.29 0)
 			(effects
@@
 			)
 		)
-		(property "MPN" "GJM0335C1E180GB01D"
+		(property "MPN" "CL10C330JB8NNNC"
 			(at 303.53 163.83 0)
 			(effects
@@
 			)
 		)
-		(property "SPN" "490-14486-1-ND"
+		(property "SPN" "1276-1070-1-ND"
 			(at 303.53 163.83 0)
 			(effects
