File: Ganglion_Sensors_01.kicad_sch (KiCad schematic)
At the start: 29 parts, among them U12 AD5621, U14 MCP6V13T, U15 MCP6001, U16 SN74LVC1G32, U17 LIS2DE12, U18 74LVC1G66, U21 74LVC1G66, U22 74LVC1G66, U23 74LVC2G00

Commit message: BOM cleanup
Parts:
- U14: value MCP6V13T -> MCP6V31T
- U15: MPN MCP6001RT-I/OTCT-ND -> MCP6001T-I/LT; SPN MCP6001RT-I/OTCT-ND -> MCP6001T-I/LTCT-ND
Changed lines of the file:
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@@
 			)
 		)
-		(property "MPN" "MCP6001RT-I/OTCT-ND"
+		(property "MPN" "MCP6001T-I/LT"
 			(at 50.8 119.38 0)
 			(effects
@@
 			)
 		)
-		(property "SPN" "MCP6001RT-I/OTCT-ND"
+		(property "SPN" "MCP6001T-I/LTCT-ND"
 			(at 50.8 119.38 0)
 			(effects
@@
 			)
 		)
-		(property "Value" "MCP6V13T"
+		(property "Value" "MCP6V31T"
 			(at 113.03 101.6 0)
 			(effects
