File: ganlion_power_01.kicad_sch (KiCad schematic)
At the start: 20 parts, among them SW5 SPDT, U10 NCP300, U11 NCP551, U9 NCP551

Commit message: BOM cleanup
Parts:
- U11, U9: value NCP551 -> TLV75730PDBVR; MPN NCP551SN30T1G -> TLV75730PDBVR; SPN NCP551SN30T1GOSCT-ND -> 296-51819-1-ND
Changed lines of the file:
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@@
 			)
 		)
-		(property "Value" "NCP551"
+		(property "Value" "TLV75730PDBVR"
 			(at 88.9 50.8 0)
 			(effects
@@
 			)
 		)
-		(property "MPN" "NCP551SN30T1G"
+		(property "MPN" "TLV75730PDBVR"
 			(at 88.9 45.72 0)
 			(effects
@@
 			)
 		)
-		(property "SPN" "NCP551SN30T1GOSCT-ND"
+		(property "SPN" "296-51819-1-ND"
 			(at 88.9 45.72 0)
 			(effects
@@
 			)
 		)
-		(property "Value" "NCP551"
+		(property "Value" "TLV75730PDBVR"
 			(at 207.01 50.8 0)
 			(effects
@@
 			)
 		)
-		(property "MPN" "NCP551SN30T1G"
+		(property "MPN" "TLV75730PDBVR"
 			(at 207.01 45.72 0)
 			(effects
@@
 			)
 		)
-		(property "SPN" "NCP551SN30T1GOSCT-ND"
+		(property "SPN" "296-51819-1-ND"
 			(at 207.01 45.72 0)
 			(effects
